File: hardware/mchair.brd (EAGLE design)
At the start: 25.6 x 53.5 mm, 120 parts, among them J1 UX60-MB-5S8, J2 JTAG-MINI, U1 STM32F769NIH6, U2 S25FS256SAGNFI00, U3 LAN8742A, U4 USB3315C, U5 MIC5503-1.8YMT-TR, U6 MT48LC16M16A2F4, U7 MPM3620GQV-P, U8 NCP186AMX330TAG, X1 G83270021, X2 DSC6101JI2A-025.0000, X3 DSC6101JI2A-024.0000

Commit message: Fix VDDDSI connection issue
Connections:
- new net N$7: U1.G13, U1.K12
- net VDD: no longer U1.G13, U1.K12
Routing:
- net N$7: track 0.00 -> 2.73 mm
- net VDD: track 76.8 -> 76.2 mm, vias 59 -> 57
Changed lines of the file:
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@@
 <?xml version="1.0" encoding="utf-8"?>
 <!DOCTYPE eagle SYSTEM "eagle.dtd">
-<eagle version="9.0.0">
+<eagle version="9.1.0">
 <drawing>
 <settings>
@@
 <layers>
 <layer number="1" name="Top" color="12" fill="1" visible="yes" active="yes"/>
-<layer number="2" name="GND" color="13" fill="1" visible="yes" active="yes"/>
-<layer number="3" name="PWR" color="4" fill="1" visible="yes" active="yes"/>
+<layer number="2" name="GND" color="13" fill="1" visible="no" active="yes"/>
+<layer number="3" name="PWR" color="4" fill="1" visible="no" active="yes"/>
 <layer number="4" name="Route4" color="1" fill="4" visible="no" active="no"/>
 <layer number="5" name="Route5" color="4" fill="4" visible="no" active="no"/>
@@
 <param name="checkStop" value="0"/>
 <param name="checkValues" value="0"/>
+<param name="checkNames" value="1"/>
+<param name="checkWireStubs" value="1"/>
+<param name="checkPolygonWidth" value="0"/>
 <param name="useDiameter" value="13"/>
 <param name="maxErrors" value="50"/>
@@
 <wire x1="10.25" y1="31.375" x2="10.6625" y2="30.9625" width="0.125" layer="1"/>
 <wire x1="10.6625" y1="30.0625" x2="10.6625" y2="30.9625" width="0.125" layer="1"/>
-<wire x1="6" y1="28.25" x2="5.875" y2="28.375" width="0.125" layer="16"/>
 <via x="5.75" y="31.5" extent="1-16" drill="0.25"/>
 <wire x1="5.875" y1="28.375" x2="5.625" y2="28.625" width="0.125" layer="16"/>
@@
 <contactref element="U1" pad="H11"/>
 <contactref element="C23" pad="1"/>
-<contactref element="U1" pad="G13"/>
-<contactref element="U1" pad="K12"/>
-<via x="9.2" y="18" extent="1-16" drill="0.25"/>
 <wire x1="7.875" y1="30.45" x2="7.475" y2="30.85" width="0.2" layer="1"/>
 <via x="7.475" y="30.85" extent="1-16" drill="0.25"/>
@@
 <wire x1="13.8" y1="15.8" x2="14" y2="15.6" width="0.2" layer="16"/>
 <via x="14" y="15.6" extent="1-16" drill="0.25"/>
-<wire x1="8.875" y1="16.725" x2="9.2" y2="17.05" width="0.2" layer="16"/>
-<wire x1="9.2" y1="17.05" x2="9.2" y2="18" width="0.2" layer="16"/>
 <wire x1="13.1875" y1="13.0375" x2="14" y2="13.85" width="0.2" layer="16"/>
 <wire x1="14" y1="13.85" x2="14" y2="14" width="0.2" layer="16"/>
@@
 <wire x1="3" y1="13.125" x2="3.24" y2="13.125" width="0.2" layer="1"/>
 <wire x1="3.24" y1="13.125" x2="3.725" y2="13.61" width="0.2" layer="1"/>
-<wire x1="8.8" y1="16" x2="9.2" y2="15.6" width="0.2" layer="1"/>
-<via x="9.2" y="15.6" extent="1-16" drill="0.25"/>
 <via x="11.6" y="18" extent="1-16" drill="0.25"/>
-<wire x1="15.3625" y1="35.7625" x2="14.0125" y2="35.7625" width="0.2" layer="1"/>
-<wire x1="14.0125" y1="35.7625" x2="14" y2="35.75" width="0.2" layer="1"/>
 <wire x1="15.35" y1="34.625" x2="15.125" y2="34.625" width="0.2" layer="1"/>
 <wire x1="15.125" y1="34.625" x2="14.625" y2="35.125" width="0.2" layer="1"/>
@@
 <wire x1="16.375" y1="35.525" x2="15.375" y2="36.525" width="0.2" layer="16"/>
 <wire x1="15.375" y1="36.525" x2="15.375" y2="36.67" width="0.2" layer="16"/>
-<wire x1="9.6" y1="18.4" x2="9.2" y2="18" width="0.2" layer="1"/>
 <wire x1="7.625" y1="4.75" x2="7.625" y2="5.375" width="0.2" layer="16"/>
 <via x="7.625" y="5.375" extent="1-16" drill="0.25"/>
@@
 <wire x1="21.7775" y1="41.04" x2="22.585" y2="41.04" width="0.2" layer="16"/>
 <wire x1="22.585" y1="41.04" x2="22.625" y2="41" width="0.2" layer="16"/>
+<wire x1="8.875" y1="16.725" x2="8.875" y2="16.875" width="0.2" layer="16"/>
+<wire x1="8.875" y1="16.875" x2="10" y2="18" width="0.2" layer="16"/>
+<wire x1="15.3625" y1="35.7625" x2="14.0375" y2="35.7625" width="0.2" layer="1"/>
+<wire x1="14.0375" y1="35.7625" x2="13.875" y2="35.6" width="0.2" layer="1"/>
 </signal>
 <signal name="USB-3.3V">
@@
 <wire x1="2.5" y1="15.415" x2="2.5" y2="39.125" width="0.125" layer="16"/>
 </signal>
+<signal name="N$7" class="1">
+<contactref element="U1" pad="G13"/>
+<contactref element="U1" pad="K12"/>
+<wire x1="9.6" y1="18.4" x2="9.2125" y2="18.0125" width="0.125" layer="1"/>
+<wire x1="9.2125" y1="16.4125" x2="8.8" y2="16" width="0.125" layer="1"/>
+<wire x1="9.2125" y1="18.0125" x2="9.2125" y2="16.4125" width="0.125" layer="1"/>
+</signal>
 </signals>
-<errors>
-</errors>
+<mfgpreviewcolors>
+<mfgpreviewcolor name="soldermaskcolor" color="0xC8008000"/>
+<mfgpreviewcolor name="silkscreencolor" color="0xFFFEFEFE"/>
+<mfgpreviewcolor name="backgroundcolor" color="0xFF282828"/>
+<mfgpreviewcolor name="coppercolor" color="0xFFFFBF00"/>
+<mfgpreviewcolor name="substratecolor" color="0xFF786E46"/>
+</mfgpreviewcolors>
 </board>
 </drawing>
