File: hardware/mchair.brd (EAGLE design)
At the start: 25.6 x 53.5 mm, 120 parts, among them J1 UX60-MB-5S8, J2 JTAG-MINI, U1 STM32F769NIH6, U2 S25FS256SAGNFI00, U3 LAN8742A, U4 USB3315C, U5 MIC5503-1.8YMT-TR, U6 MT48LC16M16A2F4, U7 MPM3620GQV-P, U8 NCP186AMX330TAG, X1 G83270021, X2 DSC6101JI2A-025.0000, X3 DSC6101JI2A-024.0000

Commit message: Move board to bare minimum for 6 layer
Routing:
- net OUT-G3: vias 2 -> 1
- net OUT-G2: vias 2 -> 1
- net OUT-G1: vias 2 -> 1
- added copper zone on layer 14, net GND
- added copper zone on layer 15, net GND
- added copper zone on layer 14, net REG-OUT
- added copper zone on layer 14, net VDD
- removed copper zone on layer 3, net GND
- removed copper zone on layer 2, net REG-OUT
- removed copper zone on layer 3, net VDD

Commit message: Start 6 layer routing
Parts:
- moved U6 0.13 mm to (10.4, 32.0)
Routing:
- net OUT-E1: track 70.5 -> 0.00 mm, vias 5 -> 0
- net OUT-E3: track 64.9 -> 0.00 mm, vias 5 -> 0
- net OUT-E2: track 64.4 -> 0.00 mm, vias 1 -> 0
- net OTG_HS-D7: track 44.4 -> 0.00 mm, vias 2 -> 0
- net OTG_HS-D3: track 44.2 -> 0.00 mm, vias 3 -> 0
- net QSPI-D2: track 42.6 -> 0.00 mm, vias 1 -> 0
- net OTG_HS-D6: track 42.5 -> 0.00 mm, vias 3 -> 0
- net OTG_HS-D5: track 42.0 -> 0.00 mm, vias 3 -> 0
- net OTG_HS-D4: track 39.7 -> 0.00 mm, vias 3 -> 0
- net QSPI-D3: track 39.6 -> 0.00 mm, vias 4 -> 0
- net OUT-B1: track 37.7 -> 0.00 mm, vias 2 -> 0
- net OUT-B5: track 37.4 -> 0.00 mm, vias 2 -> 0
- net QSPI-D0: track 35.1 -> 0.00 mm, vias 4 -> 0
- net OTG_HS-NXT: track 34.4 -> 0.00 mm, vias 3 -> 0
- net OTG_HS-STP: track 34.3 -> 0.00 mm, vias 3 -> 0
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
Commit message: continue routing breakout
Parts:
- moved C19 14.4 mm to (-4.05, 20.0)
- moved C3 4.94 mm to (8.20, 20.4), turned to 0 degrees
- moved R10 2.68 mm to (6.53, 39.3)
- moved C46 2.00 mm to (6.50, 38.5)
- moved U2 1.26 mm to (12.2, 39.8)
- moved C20 0.38 mm to (9.68, 16.4), turned to 0 degrees
- moved C12 0.10 mm to (12.4, 19.8)
- moved C5 0.10 mm to (8.54, 14.8)
Routing:
- net QSPI-D1: track 0.00 -> 50.1 mm, vias 0 -> 1
- net QSPI-CLK: track 0.00 -> 43.9 mm, vias 0 -> 1
- net QSPI-D2: track 0.00 -> 43.2 mm, vias 0 -> 1
- net QSPI-D0: track 0.00 -> 40.0 mm, vias 0 -> 1
- net QSPI-D3: track 0.00 -> 35.9 mm, vias 0 -> 1
- net QSPI-!CS: track 0.00 -> 30.8 mm, vias 0 -> 1
- net FMC-LDQM: track 0.00 -> 30.1 mm, vias 0 -> 2
- net OTG_HS-D7: track 0.00 -> 27.5 mm, vias 0 -> 1
- net FMC-SDNCAS: track 0.00 -> 26.2 mm, vias 0 -> 2
- net FMC-SDCLK: track 0.00 -> 25.0 mm
- net FMC-A0: track 0.57 -> 23.7 mm, vias 1 -> 2
- net OTG_HS-D6: track 0.00 -> 21.3 mm, vias 0 -> 1
- net OTG_HS-D5: track 0.00 -> 20.2 mm, vias 0 -> 1
- net OTG_HS-DIR: track 0.00 -> 18.5 mm
- net OTG_HS-STP: track 0.00 -> 18.3 mm
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Other:
- board text added: "mTrain v1.0"
- board text removed: "???? v1.0"

Commit message: 6 layer no DRC errors
Parts:
- moved C19 9.59 mm to (5.39, 18.4), flipped to the top, turned to 90 degrees
- moved C14 3.22 mm to (13.0, 9.47)
- moved R20 2.60 mm to (22.4, 10.2)
- moved R11 2.51 mm to (18.3, 9.00), flipped to the top
- moved R23 2.40 mm to (22.2, 4.90)
- moved R21 2.34 mm to (22.2, 2.63), turned to 90 degrees
- moved C36 2.32 mm to (18.6, 2.95)
- moved R18 2.30 mm to (22.4, 7.95), turned to 90 degrees
- moved R12 1.30 mm to (15.2, 9.43), turned to 180 degrees
- moved C29 1.03 mm to (15.7, 35.7), turned to 180 degrees
- moved R2 0.80 mm to (16.8, 17.2)
- moved U2 0.80 mm to (11.4, 39.8)
- moved R10 0.57 mm to (6.12, 38.9)
- moved C26 0.30 mm to (21.0, 10.1)
- moved C20 0.10 mm to (9.57, 16.4)
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Connections:
- net ETH-RX_N: now also JP2.18; no longer JP2.17
- net ETH-RX_P: now also JP2.17; no longer JP2.18
- net ETH-TX_N: now also JP2.20; no longer JP2.19
- net ETH-TX_P: now also JP2.19; no longer JP2.20
- net FMC-D0: now also U6.C9; no longer U6.A8
- net FMC-D10: now also U6.C1; no longer U6.D1
- net FMC-D12: now also U6.D1; no longer U6.C1
- net FMC-D13: now also U6.A2; no longer U6.B2
- net FMC-D14: now also U6.B2; no longer U6.B1
- net FMC-D15: now also U6.B1; no longer U6.A2
- net FMC-D3: now also U6.A8; no longer U6.C9
- net FMC-D4: now also U6.E9; no longer U6.C8
- net FMC-D5: now also U6.C8; no longer U6.D9
- net FMC-D7: now also U6.D9; no longer U6.E9
- net FMC-D8: now also U6.D2; no longer U6.E1
- net FMC-D9: now also U6.E1; no longer U6.D2
Routing:
- net OUT-E1: track 0.00 -> 42.5 mm, vias 0 -> 1
- net OUT-E3: track 0.00 -> 39.2 mm, vias 0 -> 2
- net OUT-E2: track 0.00 -> 38.1 mm, vias 0 -> 2
- net OUT-B5: track 0.70 -> 36.1 mm
- net OUT-B2: track 0.00 -> 28.8 mm, vias 0 -> 2
- net OUT-B1: track 0.00 -> 25.6 mm, vias 0 -> 2
- net OUT-B4: track 0.68 -> 24.3 mm, vias 1 -> 2
- net OUT-B3: track 1.57 -> 24.6 mm, vias 1 -> 2
- net ETH-RX_N: track 0.00 -> 22.7 mm
- net ETH-TX_N: track 0.00 -> 22.1 mm
- net ETH-RX_P: track 0.00 -> 22.0 mm
- net ETH-TX_P: track 0.00 -> 21.3 mm
- net OUT-C2: track 0.00 -> 19.7 mm, vias 0 -> 1
- net OUT-F1: track 0.70 -> 19.7 mm
- net OUT-D2: track 0.00 -> 18.1 mm, vias 0 -> 2
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
Commit message: v0.2 and pin numbers
Parts:
- moved R32 1.30 mm to (10.0, 0.95), flipped to the bottom, turned to 180 degrees
- moved R33 1.22 mm to (5.20, 0.93), flipped to the bottom, turned to 180 degrees
- moved D5 0.28 mm to (5.20, 0.80)
- moved D2 0.28 mm to (20.2, 0.80)
- moved D3 0.28 mm to (15.2, 0.80)
- moved D4 0.28 mm to (10.2, 0.80)
- flipped R31 to the bottom
Routing:
- net N$1: track 2.05 -> 3.75 mm
- net N$3: track 1.35 -> 2.66 mm, vias 0 -> 1
- net OUT-F4: track 15.5 -> 16.6 mm
- net LED2: track 19.5 -> 20.5 mm
- net N$2: track 1.94 -> 2.77 mm, vias 0 -> 1
- net N$4: track 1.23 -> 2.00 mm, vias 0 -> 1
- net LED4: track 26.0 -> 25.3 mm
Other:
- board text added: "GND"
- board text added: "LED1"
- board text added: "LED2"
- board text added: "LED3"
- board text added: "LED4"
- board text added: "P10"
- board text added: "P11"
- board text added: "P12"
- board text added: "P13"
- board text added: "P14"
- board text added: "P15"
- board text added: "P16"
- board text added: "P17"
- board text added: "P18"
- board text added: "P19"
- board text added: "P20"
- board text added: "P25"
- board text added: "P26"
- board text added: "P27"
- board text added: "P28"
- board text added: "P29"
- board text added: "P3"
- board text added: "P30"
- board text added: "P31"
- board text added: "P32"
- board text added: "P33"
- board text added: "P34"
- board text added: "P35"
- board text added: "P36"
- board text added: "P4"
- board text added: "P5"
- board text added: "P6"
- board text added: "P7"
- board text added: "P8"
- board text added: "P9"
- board text added: "RST"
- board text added: "RX+"
- board text added: "RX-"
- board text added: "TX+"
- board text added: "TX-"
- board text added: "VBUS"
- board text added: "VDD"
- board text added: "VIN"
- board text added: "mTrain v0.2"
- board text removed: "mTrain v1.0"
