File: hardware/mchair.sch (EAGLE design)
At the start: 119 parts, among them J1 UX60-MB-5S8, J2 JTAG-MINI, U1 STM32F769NIH6, U2 S25FS256SAGNFI00, U3 LAN8742A, U4 USB3315C, U5 MIC5503-1.8YMT-TR, U6 MT48LC16M16A2F4, U7 MPM3620GQV-P, U8 NCP186AMX330TAG, X1 G83270021, X2 DSC6101JI2A-025.0000, X3 DSC6101JI2A-024.0000

Commit message: Fix VDDDSI connection issue
Connections:
- new net N$7: U1C.VCAPDSI, U1C.VDD12DSI
- net VDD: no longer U1C.VCAPDSI, U1C.VDD12DSI
Changed lines of the file:
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@@
 <?xml version="1.0" encoding="utf-8"?>
 <!DOCTYPE eagle SYSTEM "eagle.dtd">
-<eagle version="9.0.0">
+<eagle version="9.1.0">
 <drawing>
 <settings>
@@
 <wire x1="124.46" y1="60.96" x2="124.46" y2="68.58" width="0.1524" layer="91"/>
 <junction x="124.46" y="68.58"/>
-<pinref part="U1" gate="C" pin="VDD12DSI"/>
-<wire x1="127" y1="58.42" x2="124.46" y2="58.42" width="0.1524" layer="91"/>
-<wire x1="124.46" y1="58.42" x2="124.46" y2="53.34" width="0.1524" layer="91"/>
-<pinref part="U1" gate="C" pin="VCAPDSI"/>
-<wire x1="124.46" y1="53.34" x2="127" y2="53.34" width="0.1524" layer="91"/>
-<wire x1="124.46" y1="58.42" x2="124.46" y2="60.96" width="0.1524" layer="91"/>
-<junction x="124.46" y="58.42"/>
-<junction x="124.46" y="60.96"/>
 </segment>
 <segment>
@@
 </segment>
 </net>
+<net name="N$7" class="1">
+<segment>
+<pinref part="U1" gate="C" pin="VCAPDSI"/>
+<pinref part="U1" gate="C" pin="VDD12DSI"/>
+<wire x1="127" y1="58.42" x2="124.46" y2="58.42" width="0.1524" layer="91"/>
+<wire x1="124.46" y1="58.42" x2="124.46" y2="53.34" width="0.1524" layer="91"/>
+<wire x1="124.46" y1="53.34" x2="127" y2="53.34" width="0.1524" layer="91"/>
+</segment>
+</net>

Commit message: 6 layer no DRC errors
Connections:
- net ETH-RX_N: now also JP2.18; no longer JP2.17
- net ETH-RX_P: now also JP2.17; no longer JP2.18
- net ETH-TX_N: now also JP2.20; no longer JP2.19
- net ETH-TX_P: now also JP2.19; no longer JP2.20
- net FMC-D0: now also U6.DQ3; no longer U6.DQ0
- net FMC-D10: now also U6.DQ12; no longer U6.DQ10
- net FMC-D12: now also U6.DQ10; no longer U6.DQ12
- net FMC-D13: now also U6.DQ15; no longer U6.DQ13
- net FMC-D14: now also U6.DQ13; no longer U6.DQ14
- net FMC-D15: now also U6.DQ14; no longer U6.DQ15
- net FMC-D3: now also U6.DQ0; no longer U6.DQ3
- net FMC-D4: now also U6.DQ7; no longer U6.DQ4
- net FMC-D5: now also U6.DQ4; no longer U6.DQ5
- net FMC-D7: now also U6.DQ5; no longer U6.DQ7
- net FMC-D8: now also U6.DQ9; no longer U6.DQ8
- net FMC-D9: now also U6.DQ8; no longer U6.DQ9
Changed lines of the file:
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@@
 <?xml version="1.0" encoding="utf-8"?>
 <!DOCTYPE eagle SYSTEM "eagle.dtd">
-<eagle version="9.1.0">
+<eagle version="9.1.1">
 <drawing>
 <settings>
@@
 </segment>
 </net>
-<net name="FMC-D0" class="0">
-<segment>
-<pinref part="U6" gate="G$1" pin="DQ0"/>
-<wire x1="337.82" y1="152.4" x2="340.36" y2="152.4" width="0.1524" layer="91"/>
-<label x="340.36" y="152.4" size="1.27" layer="95" xref="yes"/>
-</segment>
-</net>
 <net name="FMC-D1" class="0">
 <segment>
@@
 <net name="FMC-D3" class="0">
 <segment>
-<pinref part="U6" gate="G$1" pin="DQ3"/>
-<wire x1="337.82" y1="144.78" x2="340.36" y2="144.78" width="0.1524" layer="91"/>
-<label x="340.36" y="144.78" size="1.27" layer="95" xref="yes"/>
+<pinref part="U6" gate="G$1" pin="DQ0"/>
+<wire x1="337.82" y1="152.4" x2="340.36" y2="152.4" width="0.1524" layer="91"/>
+<label x="340.36" y="152.4" size="1.27" layer="95" xref="yes"/>
 </segment>
 </net>
-<net name="FMC-D4" class="0">
+<net name="FMC-D5" class="0">
 <segment>
 <pinref part="U6" gate="G$1" pin="DQ4"/>
@@
 </segment>
 </net>
-<net name="FMC-D5" class="0">
-<segment>
-<pinref part="U6" gate="G$1" pin="DQ5"/>
-<wire x1="337.82" y1="139.7" x2="340.36" y2="139.7" width="0.1524" layer="91"/>
-<label x="340.36" y="139.7" size="1.27" layer="95" xref="yes"/>
-</segment>
-</net>
 <net name="FMC-D6" class="0">
 <segment>
@@
 <net name="FMC-D7" class="0">
 <segment>
-<pinref part="U6" gate="G$1" pin="DQ7"/>
-<wire x1="337.82" y1="134.62" x2="340.36" y2="134.62" width="0.1524" layer="91"/>
-<label x="340.36" y="134.62" size="1.27" layer="95" xref="yes"/>
+<pinref part="U6" gate="G$1" pin="DQ5"/>
+<wire x1="337.82" y1="139.7" x2="340.36" y2="139.7" width="0.1524" layer="91"/>
+<label x="340.36" y="139.7" size="1.27" layer="95" xref="yes"/>
 </segment>
 </net>
-<net name="FMC-D8" class="0">
+<net name="FMC-D9" class="0">
 <segment>
 <pinref part="U6" gate="G$1" pin="DQ8"/>
@@
 </segment>
 </net>
-<net name="FMC-D9" class="0">
-<segment>
-<pinref part="U6" gate="G$1" pin="DQ9"/>
-<wire x1="337.82" y1="129.54" x2="340.36" y2="129.54" width="0.1524" layer="91"/>
-<label x="340.36" y="129.54" size="1.27" layer="95" xref="yes"/>
-</segment>
-</net>
 <net name="FMC-D10" class="0">
 <segment>
-<pinref part="U6" gate="G$1" pin="DQ10"/>
-<wire x1="337.82" y1="127" x2="340.36" y2="127" width="0.1524" layer="91"/>
-<label x="340.36" y="127" size="1.27" layer="95" xref="yes"/>
+<pinref part="U6" gate="G$1" pin="DQ12"/>
+<wire x1="337.82" y1="121.92" x2="340.36" y2="121.92" width="0.1524" layer="91"/>
+<label x="340.36" y="121.92" size="1.27" layer="95" xref="yes"/>
 </segment>
 </net>
@@
 </segment>
 </net>
-<net name="FMC-D12" class="0">
+<net name="FMC-D13" class="0">
 <segment>
-<pinref part="U6" gate="G$1" pin="DQ12"/>
-<wire x1="337.82" y1="121.92" x2="340.36" y2="121.92" width="0.1524" layer="91"/>
-<label x="340.36" y="121.92" size="1.27" layer="95" xref="yes"/>
+<pinref part="U6" gate="G$1" pin="DQ15"/>
+<wire x1="337.82" y1="114.3" x2="340.36" y2="114.3" width="0.1524" layer="91"/>
+<label x="340.36" y="114.3" size="1.27" layer="95" xref="yes"/>
 </segment>
 </net>
-<net name="FMC-D13" class="0">
+<net name="FMC-D14" class="0">
 <segment>
 <pinref part="U6" gate="G$1" pin="DQ13"/>
@@
 </segment>
 </net>
-<net name="FMC-D14" class="0">
-<segment>
-<pinref part="U6" gate="G$1" pin="DQ14"/>
-<wire x1="337.82" y1="116.84" x2="340.36" y2="116.84" width="0.1524" layer="91"/>
-<label x="340.36" y="116.84" size="1.27" layer="95" xref="yes"/>
-</segment>
-</net>
-<net name="FMC-D15" class="0">
-<segment>
-<pinref part="U6" gate="G$1" pin="DQ15"/>
-<wire x1="337.82" y1="114.3" x2="340.36" y2="114.3" width="0.1524" layer="91"/>
-<label x="340.36" y="114.3" size="1.27" layer="95" xref="yes"/>
-</segment>
-</net>
 <net name="FMC-A0" class="0">
 <segment>
@@
 </segment>
 </net>
+<net name="FMC-D0" class="0">
+<segment>
+<pinref part="U6" gate="G$1" pin="DQ3"/>
+<wire x1="337.82" y1="144.78" x2="340.36" y2="144.78" width="0.1524" layer="91"/>
+<label x="340.36" y="144.78" size="1.27" layer="95" xref="yes"/>
+</segment>
+</net>
+<net name="FMC-D4" class="0">
+<segment>
+<pinref part="U6" gate="G$1" pin="DQ7"/>
+<wire x1="337.82" y1="134.62" x2="340.36" y2="134.62" width="0.1524" layer="91"/>
+<label x="340.36" y="134.62" size="1.27" layer="95" xref="yes"/>
+</segment>
+</net>
+<net name="FMC-D15" class="0">
+<segment>
+<pinref part="U6" gate="G$1" pin="DQ14"/>
+<wire x1="337.82" y1="116.84" x2="340.36" y2="116.84" width="0.1524" layer="91"/>
+<label x="340.36" y="116.84" size="1.27" layer="95" xref="yes"/>
+</segment>
+</net>
+<net name="FMC-D12" class="0">
+<segment>
+<pinref part="U6" gate="G$1" pin="DQ10"/>
+<wire x1="337.82" y1="127" x2="340.36" y2="127" width="0.1524" layer="91"/>
+<label x="340.36" y="127" size="1.27" layer="95" xref="yes"/>
+</segment>
+</net>
+<net name="FMC-D8" class="0">
+<segment>
+<pinref part="U6" gate="G$1" pin="DQ9"/>
+<wire x1="337.82" y1="129.54" x2="340.36" y2="129.54" width="0.1524" layer="91"/>
+<label x="340.36" y="129.54" size="1.27" layer="95" xref="yes"/>
+</segment>
+</net>
 </nets>
 </sheet>
@@
 </segment>
 </net>
-<net name="ETH-TX_P" class="0">
+<net name="ETH-TX_N" class="0">
 <segment>
 <pinref part="JP2" gate="A" pin="20"/>
@@
 </segment>
 </net>
-<net name="ETH-TX_N" class="0">
-<segment>
-<pinref part="JP2" gate="A" pin="19"/>
-<wire x1="88.9" y1="182.88" x2="93.98" y2="182.88" width="0.1524" layer="91"/>
-<label x="93.98" y="182.88" size="1.27" layer="95" xref="yes"/>
-</segment>
-</net>
-<net name="ETH-RX_P" class="0">
+<net name="ETH-RX_N" class="0">
 <segment>
 <pinref part="JP2" gate="A" pin="18"/>
@@
 </segment>
 </net>
-<net name="ETH-RX_N" class="0">
-<segment>
-<pinref part="JP2" gate="A" pin="17"/>
-<wire x1="88.9" y1="187.96" x2="93.98" y2="187.96" width="0.1524" layer="91"/>
-<label x="93.98" y="187.96" size="1.27" layer="95" xref="yes"/>
-</segment>
-</net>
 <net name="OUT-D1" class="0">
 <segment>
@@
 </segment>
 </net>
+<net name="ETH-TX_P" class="0">
+<segment>
+<pinref part="JP2" gate="A" pin="19"/>
+<wire x1="88.9" y1="182.88" x2="93.98" y2="182.88" width="0.1524" layer="91"/>
+<label x="93.98" y="182.88" size="1.27" layer="95" xref="yes"/>
+</segment>
+</net>
+<net name="ETH-RX_P" class="0">
+<segment>
+<pinref part="JP2" gate="A" pin="17"/>
+<wire x1="88.9" y1="187.96" x2="93.98" y2="187.96" width="0.1524" layer="91"/>
+<label x="93.98" y="187.96" size="1.27" layer="95" xref="yes"/>
+</segment>
+</net>
