File: mchair.brd (EAGLE design)
At the start: 25.6 x 53.5 mm, 120 parts, among them J1 UX60-MB-5S8, J2 JTAG-MINI, U1 STM32F769NIH6, U2 S25FS256SAGNFI00, U3 LAN8742A, U4 USB3315C, U5 MIC5503-1.8YMT-TR, U6 MT48LC16M16A2F4, U7 MPM3620GQV-P, U8 NCP186AMX330TAG, X1 G83270021, X2 DSC6101JI2A-025.0000, X3 DSC6101JI2A-024.0000

Commit message: minor changes for v1.0
Parts:
- moved X3 0.32 mm to (19.3, 46.3)
- moved C34 0.23 mm to (19.7, 46.5), turned to 180 degrees
- moved X2 0.23 mm to (21.6, 7.53), turned to 0 degrees
Connections:
- net N$1 renamed LED1-PRE
- net N$2 renamed LED3-PRE
- net N$3 renamed LED2-PRE
- net N$4 renamed LED4-PRE
- net N$5 renamed LED-USB-PRE
- net N$6 renamed LED-VDD-PRE
- net N$7 renamed VDD12DSI
Other:
- board text added: "mTrain v1.0"
- board text removed: "mTrain v0.2"

Commit message: v.1
Parts:
- D6: value BLUE -> GREEN
- L1: value BLM15AG601SN1D -> BLM15
- L2: value BLM15PX121SN1D -> BLM15
- X2: value DSC6101JI2A-025.0000 -> DSC6101JI2A
- X3: value DSC6101JI2A-024.0000 -> DSC6101JI2A
