File: mchair.sch (EAGLE design)
At the start: 119 parts, among them J1 UX60-MB-5S8, J2 JTAG-MINI, U1 STM32F769NIH6, U2 S25FS256SAGNFI00, U3 LAN8742A, U4 USB3315C, U5 MIC5503-1.8YMT-TR, U6 MT48LC16M16A2F4, U7 MPM3620GQV-P, U8 NCP186AMX330TAG, X1 G83270021, X2 DSC6101JI2A-025.0000, X3 DSC6101JI2A-024.0000

Commit message: minor changes for v1.0
Connections:
- net N$1 renamed LED1-PRE
- net N$2 renamed LED3-PRE
- net N$3 renamed LED2-PRE
- net N$4 renamed LED4-PRE
- net N$5 renamed LED-USB-PRE
- net N$6 renamed LED-VDD-PRE
- net N$7 renamed VDD12DSI
Changed lines of the file:
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@@
 </segment>
 </net>
-<net name="N$7" class="1">
+<net name="VDD12DSI" class="1">
 <segment>
 <pinref part="U1" gate="C" pin="VCAPDSI"/>
@@
 </segment>
 </net>
-<net name="N$1" class="0">
+<net name="LED1-PRE" class="0">
 <segment>
 <pinref part="D2" gate="G$1" pin="A"/>
@@
 </segment>
 </net>
-<net name="N$2" class="0">
+<net name="LED3-PRE" class="0">
 <segment>
 <pinref part="D3" gate="G$1" pin="A"/>
@@
 </segment>
 </net>
-<net name="N$3" class="0">
+<net name="LED2-PRE" class="0">
 <segment>
 <pinref part="D4" gate="G$1" pin="A"/>
@@
 </segment>
 </net>
-<net name="N$4" class="0">
+<net name="LED4-PRE" class="0">
 <segment>
 <pinref part="D5" gate="G$1" pin="A"/>
@@
 </segment>
 </net>
-<net name="N$5" class="0">
+<net name="LED-USB-PRE" class="0">
 <segment>
 <pinref part="D6" gate="G$1" pin="A"/>
@@
 </segment>
 </net>
-<net name="N$6" class="0">
+<net name="LED-VDD-PRE" class="0">
 <segment>
 <pinref part="D7" gate="G$1" pin="A"/>

Commit message: v.1
Parts:
- D6: value BLUE -> GREEN; device mchair:LED-SMD-BLUE -> mchair:LED-SMD-GREEN
- L1: value BLM15AG601SN1D -> BLM15; device mchair:BLM15AG601SN1D -> mchair:BLM15
- L2: value BLM15PX121SN1D -> BLM15; device mchair:BLM15PX121SN1D -> mchair:BLM15
- X2: value DSC6101JI2A-025.0000 -> DSC6101JI2A; device mchair:DSC6101JI2A-025.0000 -> mchair:DSC6101JI2A
- X3: value DSC6101JI2A-024.0000 -> DSC6101JI2A; device mchair:DSC6101JI2A-024.0000 -> mchair:DSC6101JI2A
