File: mTrain.brd (EAGLE design)
At the start: 25.6 x 53.5 mm, 120 parts, among them J1 UX60-MB-5S8, J2 JTAG-MINI, U1 STM32F769NIH6, U2 S25FS256SAGNFI00, U3 LAN8742A, U4 USB3315C, U5 MIC5503-1.8YMT-TR, U6 MT48LC16M16A2F4, U7 MPM3620GQV-P, U8 NCP186AMX330TAG, X1 G83270021, X2 DSC6101JI2A-025.0000, X3 DSC6101JI2A-024.0000

Commit message: Renamed mchair library to mtrain
Parts:
- D1: device mchair:SOT1061 -> mTrain:SOT1061
- D2, D3, D4, D5, D6, D7: device mchair:CHIP-LED0603 -> mTrain:CHIP-LED0603
- J1: device mchair:UX60-MB-5S8 -> mTrain:UX60-MB-5S8
- J2: device mchair:FTSH-105-01-F-D-K -> mTrain:FTSH-105-01-F-D-K
- JP1, JP2: device mchair:1X20 -> mTrain:1X20
- L1, L2: device mchair:0402 -> mTrain:0402
- S1: device mchair:EVQ-P7C01P -> mTrain:EVQ-P7C01P
- S2: device mchair:EVP-BFAC1A000 -> mTrain:EVP-BFAC1A000
- U1: device mchair:TFBGA216 -> mTrain:TFBGA216
- U2: device mchair:WSON8 -> mTrain:WSON8
- U3, U4: device mchair:VQFN24 -> mTrain:VQFN24
- U5: device mchair:MIC5503-1.8YMT-TR -> mTrain:MIC5503-1.8YMT-TR
- U6: device mchair:VFBGA54 -> mTrain:VFBGA54
- U7: device mchair:MPM3620GQV-P -> mTrain:MPM3620GQV-P
- U8: device mchair:XDFN8 -> mTrain:XDFN8
- X1: device mchair:G83270021 -> mTrain:G83270021
- X2, X3: device mchair:DSC6101JI2A -> mTrain:DSC6101JI2A
Other:
- board text added: ">VERSION"
- board text added: "mTrain"
- board text removed: "mTrain v1.0"
