File: mTrain.sch (EAGLE design)
At the start: 119 parts, among them J1 UX60-MB-5S8, J2 JTAG-MINI, U1 STM32F769NIH6, U2 S25FS256SAGNFI00, U3 LAN8742A, U4 USB3315C, U5 MIC5503-1.8YMT-TR, U6 MT48LC16M16A2F4, U7 MPM3620GQV-P, U8 NCP186AMX330TAG, X1 G83270021, X2 DSC6101JI2A-025.0000, X3 DSC6101JI2A-024.0000

Commit message: Renamed mchair library to mtrain
Parts:
- D1: device mchair:PMEG3020CPA,115 -> mTrain:PMEG3020CPA,115
- D2, D3, D4, D5, D6: device mchair:LED-SMD-BLUE -> mTrain:LED-SMD-BLUE
- D7: device mchair:LED-SMD-GREEN -> mTrain:LED-SMD-GREEN
- J1: device mchair:UX60-MB-5S8 -> mTrain:UX60-MB-5S8
- J2: device mchair:JTAG-MINI -> mTrain:JTAG-MINI
- JP1, JP2: device mchair:PINHD-1X20 -> mTrain:PINHD-1X20
- L1: device mchair:BLM15AG601SN1D -> mTrain:BLM15AG601SN1D
- L2: device mchair:BLM15PX121SN1D -> mTrain:BLM15PX121SN1D
- S1: device mchair:EVQ-P7C01P -> mTrain:EVQ-P7C01P
- S2: device mchair:EVP-BFAC1A000 -> mTrain:EVP-BFAC1A000
- U1: device mchair:STM32F769NIH6 -> mTrain:STM32F769NIH6
- U2: device mchair:S25FS256SAGNFI00 -> mTrain:S25FS256SAGNFI00
- U3: device mchair:LAN8742A -> mTrain:LAN8742A
- U4: device mchair:USB3315C -> mTrain:USB3315C
- U5: device mchair:MIC5503-1.8YMT-TR -> mTrain:MIC5503-1.8YMT-TR
- U6: device mchair:MT48LC16M16A2F4 -> mTrain:MT48LC16M16A2F4
- U7: device mchair:MPM3620GQV-P -> mTrain:MPM3620GQV-P
- U8: device mchair:NCP186AMX330TAG -> mTrain:NCP186AMX330TAG
- X1: device mchair:G83270021 -> mTrain:G83270021
- X2: device mchair:DSC6101JI2A-025.0000 -> mTrain:DSC6101JI2A-025.0000
- X3: device mchair:DSC6101JI2A-024.0000 -> mTrain:DSC6101JI2A-024.0000
